File: hardware/eagle/WearablesVCNL4020small.sch (EAGLE design)
At the start: 11 parts

Commit message: Add files via upload
Other:
- note added: "Flex Cable Pads"
- moved on the sheet: 3V3, GND, INT, SCL, SDA
Changed lines of the file:
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@@
 <plain>
 <text x="5.08" y="48.26" size="1.778" layer="95">VCNL 4020</text>
+<text x="58.42" y="76.2" size="1.778" layer="95">Flex Cable Pads</text>
 </plain>
 <instances>
@@
 <instance part="U$1" gate="G$1" x="12.7" y="68.58"/>
 <instance part="GND3" gate="1" x="50.8" y="68.58"/>
-<instance part="GND" gate="G$1" x="76.2" y="101.6" rot="R270"/>
-<instance part="3V3" gate="G$1" x="76.2" y="96.52" rot="R270"/>
-<instance part="INT" gate="G$1" x="76.2" y="91.44" rot="R270"/>
-<instance part="SCL" gate="G$1" x="76.2" y="86.36" rot="R270"/>
-<instance part="SDA" gate="G$1" x="76.2" y="81.28" rot="R270"/>
+<instance part="GND" gate="G$1" x="76.2" y="96.52" rot="R270"/>
+<instance part="3V3" gate="G$1" x="76.2" y="101.6" rot="R270"/>
+<instance part="INT" gate="G$1" x="76.2" y="86.36" rot="R270"/>
+<instance part="SCL" gate="G$1" x="76.2" y="81.28" rot="R270"/>
+<instance part="SDA" gate="G$1" x="76.2" y="91.44" rot="R270"/>
 </instances>
 <busses>
@@
 </segment>
 <segment>
-<label x="58.42" y="101.6" size="1.778" layer="95" rot="R180" xref="yes"/>
-<wire x1="58.42" y1="101.6" x2="73.66" y2="101.6" width="0.1524" layer="91"/>
+<label x="58.42" y="96.52" size="1.778" layer="95" rot="R180" xref="yes"/>
+<wire x1="58.42" y1="96.52" x2="73.66" y2="96.52" width="0.1524" layer="91"/>
 <pinref part="GND" gate="G$1" pin="PP"/>
 </segment>
@@
 </segment>
 <segment>
-<label x="58.42" y="96.52" size="1.778" layer="95" rot="R180" xref="yes"/>
-<wire x1="58.42" y1="96.52" x2="73.66" y2="96.52" width="0.1524" layer="91"/>
+<label x="58.42" y="101.6" size="1.778" layer="95" rot="R180" xref="yes"/>
+<wire x1="58.42" y1="101.6" x2="73.66" y2="101.6" width="0.1524" layer="91"/>
 <pinref part="3V3" gate="G$1" pin="PP"/>
 </segment>
@@
 </segment>
 <segment>
-<wire x1="73.66" y1="81.28" x2="58.42" y2="81.28" width="0.1524" layer="91"/>
-<label x="58.42" y="81.28" size="1.778" layer="95" rot="R180" xref="yes"/>
+<wire x1="73.66" y1="91.44" x2="58.42" y2="91.44" width="0.1524" layer="91"/>
+<label x="58.42" y="91.44" size="1.778" layer="95" rot="R180" xref="yes"/>
 <pinref part="SDA" gate="G$1" pin="PP"/>
 </segment>
@@
 </segment>
 <segment>
-<label x="58.42" y="86.36" size="1.778" layer="95" rot="R180" xref="yes"/>
-<wire x1="58.42" y1="86.36" x2="73.66" y2="86.36" width="0.1524" layer="91"/>
+<label x="58.42" y="81.28" size="1.778" layer="95" rot="R180" xref="yes"/>
+<wire x1="58.42" y1="81.28" x2="73.66" y2="81.28" width="0.1524" layer="91"/>
 <pinref part="SCL" gate="G$1" pin="PP"/>
 </segment>
@@
 <net name="INT" class="0">
 <segment>
-<label x="58.42" y="91.44" size="1.778" layer="95" rot="R180" xref="yes"/>
-<wire x1="73.66" y1="91.44" x2="58.42" y2="91.44" width="0.1524" layer="91"/>
+<label x="58.42" y="86.36" size="1.778" layer="95" rot="R180" xref="yes"/>
+<wire x1="73.66" y1="86.36" x2="58.42" y2="86.36" width="0.1524" layer="91"/>
 <pinref part="INT" gate="G$1" pin="PP"/>
 </segment>

Commit message: updated schematics and board files.
Parts:
- R1: value 10 -> 10R
Other:
- moved on the sheet: 3V3, C1, C2, GND, INT, R1, SCL, SDA
